Commit message: fix marvin and add pm01

File: Marvin_M6_S_CCS_696_V4.0/robot.urdf (robot description, URDF)
Before this commit: robot Marvin_M6_S_CCS_696_V4.0, 21 links, 20 joints
Links:
- link base_link: geometry collision mesh filename=collision/base_link.obj; visual mesh filename=visual/glb/base_link.glb
- link elbow_pitch_l_j3_link: geometry collision mesh filename=collision/elbow_pitch_l_j3_link.obj; visual mesh filename=visual/glb/elbow_pitch_l_j3_link.glb
- link elbow_pitch_r_j3_link: geometry collision mesh filename=collision/elbow_pitch_r_j3_link.obj; visual mesh filename=visual/glb/elbow_pitch_r_j3_link.glb
- link elbow_yaw_l_j4_link: geometry collision mesh filename=collision/elbow_yaw_l_j4_link.obj; visual mesh filename=visual/glb/elbow_yaw_l_j4_link.glb
- link elbow_yaw_r_j4_link: geometry collision mesh filename=collision/elbow_yaw_r_j4_link.obj; visual mesh filename=visual/glb/elbow_yaw_r_j4_link.glb
- link left_arm_base: geometry collision mesh filename=collision/left_arm_base.obj; visual mesh filename=visual/glb/left_arm_base.glb
- link left_ee: mass 0 -> None; geometry 
- link right_arm_base: geometry collision mesh filename=collision/right_arm_base.obj; visual mesh filename=visual/glb/right_arm_base.glb
- link right_ee: mass 0 -> None; geometry 
- link shoulder_pitch_l_j1_link: geometry collision mesh filename=collision/shoulder_pitch_l_j1_link.obj; visual mesh filename=visual/glb/shoulder_pitch_l_j1_link.glb
- link shoulder_pitch_r_j1_link: geometry collision mesh filename=collision/shoulder_pitch_r_j1_link.obj; visual mesh filename=visual/glb/shoulder_pitch_r_j1_link.glb
- link shoulder_roll_l_j2_link: geometry collision mesh filename=collision/shoulder_roll_l_j2_link.obj; visual mesh filename=visual/glb/shoulder_roll_l_j2_link.glb
- link shoulder_roll_r_j2_link: geometry collision mesh filename=collision/shoulder_roll_r_j2_link.obj; visual mesh filename=visual/glb/shoulder_roll_r_j2_link.glb
- link torso_base: geometry collision mesh filename=collision/torso_base.obj; visual mesh filename=visual/glb/torso_base.glb
- link wrist_pitch_l_j5_link: geometry collision mesh filename=collision/wrist_pitch_l_j5_link.obj; visual mesh filename=visual/glb/wrist_pitch_l_j5_link.glb
- link wrist_pitch_r_j5_link: geometry collision mesh filename=collision/wrist_pitch_r_j5_link.obj; visual mesh filename=visual/glb/wrist_pitch_r_j5_link.glb
- link wrist_roll_l_j7_link: geometry collision mesh filename=collision/wrist_roll_l_j7_link.obj; visual mesh filename=visual/glb/wrist_roll_l_j7_link.glb
- link wrist_roll_r_j7_link: geometry collision mesh filename=collision/wrist_roll_r_j7_link.obj; visual mesh filename=visual/glb/wrist_roll_r_j7_link.glb
- link wrist_yaw_l_j6_link: geometry collision mesh filename=collision/wrist_yaw_l_j6_link.obj; visual mesh filename=visual/glb/wrist_yaw_l_j6_link.glb
- link wrist_yaw_r_j6_link: geometry collision mesh filename=collision/wrist_yaw_r_j6_link.obj; visual mesh filename=visual/glb/wrist_yaw_r_j6_link.glb
Joints:
- joint TORSO_TO_LEFT_ARM_CONNECTOR: origin xyz=0 0.037 0.140 rpy=-1.5708 0 0 -> xyz=0 0.037 0 rpy=-1.5708 0 0
- joint TORSO_TO_RIGHT_ARM_CONNECTOR: origin xyz=0 -0.037 0.140 rpy=1.5708 0 0 -> xyz=0 -0.037 0 rpy=1.5708 0 0
- joint UPPER_BODY_BASE: origin xyz=0 0 0 rpy=0 0 0 -> xyz=0 0 0.140 rpy=0 0 0

File: Marvin_M6_S_CCS_696_V4.0/torso.urdf (robot description, URDF)
Before this commit: robot Marvin_M6_S_CCS_696_V4.0_torso, 3 links, 2 joints
Joints:
- joint UPPER_BODY_BASE: origin xyz=0 0 0 rpy=0 0 0 -> xyz=0 0 0.140 rpy=0 0 0
