Commit message: add robots

File: Marvin_M6_S_CCS_696_V4.0/left_arm.urdf (robot description, URDF)
Before this commit: robot Marvin_M6_S_CCS_696_V4.0_left_arm, 9 links, 8 joints
Links:
- link elbow_pitch_l_j3_link: geometry collision mesh filename=collision/elbow_pitch_l_j3_link.obj; visual mesh filename=visual/glb/elbow_pitch_l_j3_link.glb
- link elbow_yaw_l_j4_link: geometry collision mesh filename=collision/elbow_yaw_l_j4_link.obj; visual mesh filename=visual/glb/elbow_yaw_l_j4_link.glb
- link left_arm_base: mass 1.1962 -> None; geometry 
- link left_ee: mass 0 -> None; geometry 
- link shoulder_pitch_l_j1_link: geometry collision mesh filename=collision/shoulder_pitch_l_j1_link.obj; visual mesh filename=visual/glb/shoulder_pitch_l_j1_link.glb
- link shoulder_roll_l_j2_link: geometry collision mesh filename=collision/shoulder_roll_l_j2_link.obj; visual mesh filename=visual/glb/shoulder_roll_l_j2_link.glb
- link wrist_pitch_l_j5_link: geometry collision mesh filename=collision/wrist_pitch_l_j5_link.obj; visual mesh filename=visual/glb/wrist_pitch_l_j5_link.glb
- link wrist_roll_l_j7_link: geometry collision mesh filename=collision/wrist_roll_l_j7_link.obj; visual mesh filename=visual/glb/wrist_roll_l_j7_link.glb
- link wrist_yaw_l_j6_link: geometry collision mesh filename=collision/wrist_yaw_l_j6_link.obj; visual mesh filename=visual/glb/wrist_yaw_l_j6_link.glb
Joints:
- joint ELBOW_PITCH_L_J3: limit lower=-3.1067 upper=3.1067 effort=66 velocity=3.1416 -> lower=-3.1066860685499065 upper=3.1066860685499065 effort=66 velocity=3.141592653589793; origin xyz=0 0.287 0 rpy=-1.5708 0 0 -> xyz=0 0.287 0 rpy=-1.5707963267948966 0 0
- joint ELBOW_YAW_L_J4: limit lower=-2.5307 upper=1.0472 effort=66 velocity=3.1416 -> lower=-2.530727415391778 upper=1.0471975511965976 effort=66 velocity=3.141592653589793; origin xyz=0.018 0 0 rpy=-1.5708 0 3.1416 -> xyz=0.018 0 0 rpy=-1.5707963267948966 0 3.141592653589793
- joint LEFT_EE: origin xyz=0 -0.095 0 rpy=1.5708 -1.5708 0 -> xyz=0 -0.095 0 rpy=1.5707963267948966 -1.5707963267948966 0
- joint SHOULDER_PITCH_L_J1: limit lower=-3.1067 upper=3.1067 effort=108 velocity=3.1416 -> lower=-3.1066860685499065 upper=3.1066860685499065 effort=108 velocity=3.141592653589793; origin xyz=0 0 0.1745 rpy=0 0 0 -> xyz=0.2215 2.9142E-05 1.121 rpy=-1.5707963267948966 0 -1.5707963267948966
- joint SHOULDER_ROLL_L_J2: limit lower=-2.0944 upper=2.0944 effort=108 velocity=3.1416 -> lower=-2.0943951023931953 upper=2.0943951023931953 effort=108 velocity=3.141592653589793; origin xyz=0 0 0 rpy=1.5708 0 0 -> xyz=0 0 0 rpy=1.5707963267948966 0 0
- joint WRIST_PITCH_L_J5: limit lower=-3.1067 upper=3.1067 effort=18 velocity=3.1416 -> lower=-3.1066860685499065 upper=3.1066860685499065 effort=18 velocity=3.141592653589793; origin xyz=0.018 -0.314 0 rpy=-1.5708 0 3.1416 -> xyz=0.018 -0.314 0 rpy=-1.5707963267948966 0 3.141592653589793
- joint WRIST_ROLL_L_J7: limit lower=-1.5708 upper=1.5708 effort=18 velocity=3.1416 -> lower=-1.5707963267948966 upper=1.5707963267948966 effort=18 velocity=3.141592653589793; origin xyz=0 0 0 rpy=1.5708 -1.5708 0 -> xyz=0 0 0 rpy=1.5707963267948966 -1.5707963267948966 0
- joint WRIST_YAW_L_J6: limit lower=-1.0472 upper=1.0472 effort=18 velocity=3.1416 -> lower=-1.0471975511965976 upper=1.0471975511965976 effort=18 velocity=3.141592653589793; origin xyz=0 0 0 rpy=1.5708 -1.5708 0 -> xyz=0 0 0 rpy=1.5707963267948966 -1.5707963267948966 0

File: Marvin_M6_S_CCS_696_V4.0/right_arm.urdf (robot description, URDF)
Before this commit: robot Marvin_M6_S_CCS_696_V4.0_right_arm, 9 links, 8 joints
Links:
- link elbow_pitch_r_j3_link: geometry collision mesh filename=collision/elbow_pitch_r_j3_link.obj; visual mesh filename=visual/glb/elbow_pitch_r_j3_link.glb
- link elbow_yaw_r_j4_link: geometry collision mesh filename=collision/elbow_yaw_r_j4_link.obj; visual mesh filename=visual/glb/elbow_yaw_r_j4_link.glb
- link right_arm_base: mass 1.1962 -> None; geometry 
- link right_ee: mass 0 -> None; geometry 
- link shoulder_pitch_r_j1_link: geometry collision mesh filename=collision/shoulder_pitch_r_j1_link.obj; visual mesh filename=visual/glb/shoulder_pitch_r_j1_link.glb
- link shoulder_roll_r_j2_link: geometry collision mesh filename=collision/shoulder_roll_r_j2_link.obj; visual mesh filename=visual/glb/shoulder_roll_r_j2_link.glb
- link wrist_pitch_r_j5_link: geometry collision mesh filename=collision/wrist_pitch_r_j5_link.obj; visual mesh filename=visual/glb/wrist_pitch_r_j5_link.glb
- link wrist_roll_r_j7_link: geometry collision mesh filename=collision/wrist_roll_r_j7_link.obj; visual mesh filename=visual/glb/wrist_roll_r_j7_link.glb
- link wrist_yaw_r_j6_link: geometry collision mesh filename=collision/wrist_yaw_r_j6_link.obj; visual mesh filename=visual/glb/wrist_yaw_r_j6_link.glb
Joints:
- joint ELBOW_PITCH_R_J3: limit lower=-3.1067 upper=3.1067 effort=66 velocity=3.1416 -> lower=-3.1066860685499065 upper=3.1066860685499065 effort=66 velocity=3.141592653589793; origin xyz=0 0.287 0 rpy=-1.5708 0 0 -> xyz=0 0.287 0 rpy=-1.5707963267948966 0 0
- joint ELBOW_YAW_R_J4: limit lower=-2.5307 upper=1.0472 effort=66 velocity=3.1416 -> lower=-2.530727415391778 upper=1.0471975511965976 effort=66 velocity=3.141592653589793; origin xyz=0.018 0 0 rpy=-1.5708 0 3.1416 -> xyz=0.018 0 0 rpy=-1.5707963267948966 0 3.141592653589793
- joint RIGHT_EE: origin xyz=0 -0.095 0 rpy=1.5708 -1.5708 0 -> xyz=0 -0.095 0 rpy=1.5707963267948966 -1.5707963267948966 0
- joint SHOULDER_PITCH_R_J1: limit lower=-3.1067 upper=3.1067 effort=108 velocity=3.1416 -> lower=-3.1066860685499065 upper=3.1066860685499065 effort=108 velocity=3.141592653589793; origin xyz=0 0 0.1745 rpy=0 0 0 -> xyz=-0.2215 2.9142E-05 1.121 rpy=1.5707963267948966 0 -1.5707963267948966
- joint SHOULDER_ROLL_R_J2: limit lower=-2.0944 upper=2.0944 effort=108 velocity=3.1416 -> lower=-2.0943951023931953 upper=2.0943951023931953 effort=108 velocity=3.141592653589793; origin xyz=0 0 0 rpy=1.5708 0 0 -> xyz=0 0 0 rpy=1.5707963267948966 0 0
- joint WRIST_PITCH_R_J5: limit lower=-3.1067 upper=3.1067 effort=18 velocity=3.1416 -> lower=-3.1066860685499065 upper=3.1066860685499065 effort=18 velocity=3.141592653589793; origin xyz=0.018 -0.314 0 rpy=-1.5708 0 3.1416 -> xyz=0.018 -0.314 0 rpy=-1.5707963267948966 0 3.141592653589793
- joint WRIST_ROLL_R_J7: limit lower=-1.5708 upper=1.5708 effort=18 velocity=3.1416 -> lower=-1.5707963267948966 upper=1.5707963267948966 effort=18 velocity=3.141592653589793; origin xyz=0 0 0 rpy=1.5708 -1.5708 0 -> xyz=0 0 0 rpy=1.5707963267948966 -1.5707963267948966 0
- joint WRIST_YAW_R_J6: limit lower=-1.0472 upper=1.0472 effort=18 velocity=3.1416 -> lower=-1.0471975511965976 upper=1.0471975511965976 effort=18 velocity=3.141592653589793; origin xyz=0 0 0 rpy=1.5708 -1.5708 0 -> xyz=0 0 0 rpy=1.5707963267948966 -1.5707963267948966 0

File: Marvin_M6_S_CCS_696_V4.0/robot.urdf (robot description, URDF)
Before this commit: robot Marvin_M6_S_CCS_696_V4.0, 21 links, 20 joints
Links:
- removed link torso_base
- link base_link: mass 74.515 -> 63.8
- link left_arm_base: mass 1.1962 -> None; geometry 
- link right_arm_base: mass 1.1962 -> None; geometry 
Joints:
- removed joint BASE_LINK_TO_TORSO_CONNECTOR
- joint ELBOW_PITCH_L_J3: limit lower=-3.1067 upper=3.1067 effort=66 velocity=3.1416 -> lower=-3.1066860685499065 upper=3.1066860685499065 effort=66 velocity=3.141592653589793; origin xyz=0 0.287 0 rpy=-1.5708 0 0 -> xyz=0 0.287 0 rpy=-1.5707963267948966 0 0
- joint ELBOW_PITCH_R_J3: limit lower=-3.1067 upper=3.1067 effort=66 velocity=3.1416 -> lower=-3.1066860685499065 upper=3.1066860685499065 effort=66 velocity=3.141592653589793; origin xyz=0 0.287 0 rpy=-1.5708 0 0 -> xyz=0 0.287 0 rpy=-1.5707963267948966 0 0
- joint ELBOW_YAW_L_J4: limit lower=-2.5307 upper=1.0472 effort=66 velocity=3.1416 -> lower=-2.530727415391778 upper=1.0471975511965976 effort=66 velocity=3.141592653589793; origin xyz=0.018 0 0 rpy=-1.5708 0 3.1416 -> xyz=0.018 0 0 rpy=-1.5707963267948966 0 3.141592653589793
- joint ELBOW_YAW_R_J4: limit lower=-2.5307 upper=1.0472 effort=66 velocity=3.1416 -> lower=-2.530727415391778 upper=1.0471975511965976 effort=66 velocity=3.141592653589793; origin xyz=0.018 0 0 rpy=-1.5708 0 3.1416 -> xyz=0.018 0 0 rpy=-1.5707963267948966 0 3.141592653589793
- joint LEFT_EE: origin xyz=0 -0.095 0 rpy=1.5708 -1.5708 0 -> xyz=0 -0.095 0 rpy=1.5707963267948966 -1.5707963267948966 0
- joint RIGHT_EE: origin xyz=0 -0.095 0 rpy=1.5708 -1.5708 0 -> xyz=0 -0.095 0 rpy=1.5707963267948966 -1.5707963267948966 0
- joint SHOULDER_PITCH_L_J1: limit lower=-3.1067 upper=3.1067 effort=108 velocity=3.1416 -> lower=-3.1066860685499065 upper=3.1066860685499065 effort=108 velocity=3.141592653589793; origin xyz=0 0 0.1745 rpy=0 0 0 -> xyz=0.2215 2.9142E-05 1.121 rpy=-1.5707963267948966 0 -1.5707963267948966
- joint SHOULDER_PITCH_R_J1: limit lower=-3.1067 upper=3.1067 effort=108 velocity=3.1416 -> lower=-3.1066860685499065 upper=3.1066860685499065 effort=108 velocity=3.141592653589793; origin xyz=0 0 0.1745 rpy=0 0 0 -> xyz=-0.2215 2.9142E-05 1.121 rpy=1.5707963267948966 0 -1.5707963267948966
- joint SHOULDER_ROLL_L_J2: limit lower=-2.0944 upper=2.0944 effort=108 velocity=3.1416 -> lower=-2.0943951023931953 upper=2.0943951023931953 effort=108 velocity=3.141592653589793; origin xyz=0 0 0 rpy=1.5708 0 0 -> xyz=0 0 0 rpy=1.5707963267948966 0 0
- joint SHOULDER_ROLL_R_J2: limit lower=-2.0944 upper=2.0944 effort=108 velocity=3.1416 -> lower=-2.0943951023931953 upper=2.0943951023931953 effort=108 velocity=3.141592653589793; origin xyz=0 0 0 rpy=1.5708 0 0 -> xyz=0 0 0 rpy=1.5707963267948966 0 0
- joint TORSO_TO_LEFT_ARM_CONNECTOR: axis 0 0 0 -> (none); origin xyz=0 0.037 0 rpy=-1.5708 0 0 -> xyz=2.9142E-05 0 -1.121 rpy=0 0 1.5707963267948966
- joint TORSO_TO_RIGHT_ARM_CONNECTOR: axis 0 0 0 -> (none); origin xyz=0 -0.037 0 rpy=1.5708 0 0 -> xyz=2.9142E-05 0 -1.121 rpy=0 0 1.5707963267948966
- joint UPPER_BODY_BASE: origin xyz=0 0 0.140 rpy=0 0 0 -> xyz=-2.9142E-05 0 1.121 rpy=0 0 0; parent torso_base -> base_link
- joint WRIST_PITCH_L_J5: limit lower=-3.1067 upper=3.1067 effort=18 velocity=3.1416 -> lower=-3.1066860685499065 upper=3.1066860685499065 effort=18 velocity=3.141592653589793; origin xyz=0.018 -0.314 0 rpy=-1.5708 0 3.1416 -> xyz=0.018 -0.314 0 rpy=-1.5707963267948966 0 3.141592653589793
- joint WRIST_PITCH_R_J5: limit lower=-3.1067 upper=3.1067 effort=18 velocity=3.1416 -> lower=-3.1066860685499065 upper=3.1066860685499065 effort=18 velocity=3.141592653589793; origin xyz=0.018 -0.314 0 rpy=-1.5708 0 3.1416 -> xyz=0.018 -0.314 0 rpy=-1.5707963267948966 0 3.141592653589793
- joint WRIST_ROLL_L_J7: limit lower=-1.5708 upper=1.5708 effort=18 velocity=3.1416 -> lower=-1.5707963267948966 upper=1.5707963267948966 effort=18 velocity=3.141592653589793; origin xyz=0 0 0 rpy=1.5708 -1.5708 0 -> xyz=0 0 0 rpy=1.5707963267948966 -1.5707963267948966 0
- joint WRIST_ROLL_R_J7: limit lower=-1.5708 upper=1.5708 effort=18 velocity=3.1416 -> lower=-1.5707963267948966 upper=1.5707963267948966 effort=18 velocity=3.141592653589793; origin xyz=0 0 0 rpy=1.5708 -1.5708 0 -> xyz=0 0 0 rpy=1.5707963267948966 -1.5707963267948966 0
- joint WRIST_YAW_L_J6: limit lower=-1.0472 upper=1.0472 effort=18 velocity=3.1416 -> lower=-1.0471975511965976 upper=1.0471975511965976 effort=18 velocity=3.141592653589793; origin xyz=0 0 0 rpy=1.5708 -1.5708 0 -> xyz=0 0 0 rpy=1.5707963267948966 -1.5707963267948966 0
- joint WRIST_YAW_R_J6: limit lower=-1.0472 upper=1.0472 effort=18 velocity=3.1416 -> lower=-1.0471975511965976 upper=1.0471975511965976 effort=18 velocity=3.141592653589793; origin xyz=0 0 0 rpy=1.5708 -1.5708 0 -> xyz=0 0 0 rpy=1.5707963267948966 -1.5707963267948966 0

File: Marvin_M6_S_CCS_696_V4.0/torso.urdf (robot description, URDF)
Before this commit: robot Marvin_M6_S_CCS_696_V4.0_torso, 3 links, 2 joints
Links:
- removed link torso_base
- link base_link: mass 74.515 -> 63.8; geometry collision mesh filename=collision/base_link.obj; visual mesh filename=visual/glb/base_link.glb
Joints:
- removed joint BASE_LINK_TO_TORSO_CONNECTOR
- joint UPPER_BODY_BASE: origin xyz=0 0 0.140 rpy=0 0 0 -> xyz=-2.9142E-05 0 1.121 rpy=0 0 0; parent torso_base -> base_link
