Commit message: standardize humanoid assets and previews

File: Dexforce_W1_V3/robot_with_ee.urdf (robot description, URDF)
Before this commit: robot robot_with_ee__v030__[Arms-anthropomorphic], 30 links, 29 joints
Links:
- added link left_base_link
- added link left_base_offset
- added link left_connector_link; collision mesh filename=collision/left_hand/connector_link.obj; visual mesh filename=visual/left_hand/connector_link.glb
- added link left_hand_base_link, mass 0.427; collision mesh filename=collision/left_hand/hand_base_link.obj; visual mesh filename=visual/left_hand/hand_base_link.glb
- added link left_if_dip_link, mass 0.011; collision mesh filename=collision/left_hand/if_dip_link.obj; visual mesh filename=visual/left_hand/if_dip_link.glb
- added link left_if_mcp_pitch_link, mass 0.008; collision mesh filename=collision/left_hand/if_mcp_pitch_link.obj; visual mesh filename=visual/left_hand/if_mcp_pitch_link.glb
- added link left_lf_dip_link, mass 0.008; collision mesh filename=collision/left_hand/lf_dip_link.obj; visual mesh filename=visual/left_hand/lf_dip_link.glb
- added link left_lf_mcp_pitch_link, mass 0.008; collision mesh filename=collision/left_hand/lf_mcp_pitch_link.obj; visual mesh filename=visual/left_hand/lf_mcp_pitch_link.glb
- added link left_mf_dip_link, mass 0.011; collision mesh filename=collision/left_hand/mf_dip_link.obj; visual mesh filename=visual/left_hand/mf_dip_link.glb
- added link left_mf_mcp_pitch_link, mass 0.011; collision mesh filename=collision/left_hand/mf_mcp_pitch_link.obj; visual mesh filename=visual/left_hand/mf_mcp_pitch_link.glb
- added link left_rf_dip_link, mass 0.008; collision mesh filename=collision/left_hand/rf_dip_link.obj; visual mesh filename=visual/left_hand/rf_dip_link.glb
- added link left_rf_mcp_pitch_link, mass 0.011; collision mesh filename=collision/left_hand/rf_mcp_pitch_link.obj; visual mesh filename=visual/left_hand/rf_mcp_pitch_link.glb
- added link left_t_cmc_yaw_link, mass 0.005; collision mesh filename=collision/left_hand/t_cmc_yaw_link.obj; visual mesh filename=visual/left_hand/t_cmc_yaw_link.glb
- added link left_t_mcp_link, mass 0.04; collision mesh filename=collision/left_hand/t_mcp_link.obj; visual mesh filename=visual/left_hand/t_mcp_link.glb
- added link right_base_link
- added link right_base_offset
- added link right_connector_link; collision mesh filename=collision/right_hand/connector_link.obj; visual mesh filename=visual/right_hand/connector_link.glb
- added link right_hand_base_link, mass 0.427; collision mesh filename=collision/right_hand/hand_base_link.obj; visual mesh filename=visual/right_hand/hand_base_link.glb
- added link right_if_dip_link, mass 0.011; collision mesh filename=collision/right_hand/if_dip_link.obj; visual mesh filename=visual/right_hand/if_dip_link.glb
- added link right_if_mcp_pitch_link, mass 0.008; collision mesh filename=collision/right_hand/if_mcp_pitch_link.obj; visual mesh filename=visual/right_hand/if_mcp_pitch_link.glb
- added link right_lf_dip_link, mass 0.008; collision mesh filename=collision/right_hand/lf_dip_link.obj; visual mesh filename=visual/right_hand/lf_dip_link.glb
- added link right_lf_mcp_pitch_link, mass 0.008; collision mesh filename=collision/right_hand/lf_mcp_pitch_link.obj; visual mesh filename=visual/right_hand/lf_mcp_pitch_link.glb
- added link right_mf_dip_link, mass 0.011; collision mesh filename=collision/right_hand/mf_dip_link.obj; visual mesh filename=visual/right_hand/mf_dip_link.glb
- added link right_mf_mcp_pitch_link, mass 0.011; collision mesh filename=collision/right_hand/mf_mcp_pitch_link.obj; visual mesh filename=visual/right_hand/mf_mcp_pitch_link.glb
- added link right_rf_dip_link, mass 0.008; collision mesh filename=collision/right_hand/rf_dip_link.obj; visual mesh filename=visual/right_hand/rf_dip_link.glb
- added link right_rf_mcp_pitch_link, mass 0.011; collision mesh filename=collision/right_hand/rf_mcp_pitch_link.obj; visual mesh filename=visual/right_hand/rf_mcp_pitch_link.glb
- added link right_t_cmc_yaw_link, mass 0.005; collision mesh filename=collision/right_hand/t_cmc_yaw_link.obj; visual mesh filename=visual/right_hand/t_cmc_yaw_link.glb
- added link right_t_mcp_link, mass 0.04; collision mesh filename=collision/right_hand/t_mcp_link.obj; visual mesh filename=visual/right_hand/t_mcp_link.glb
Joints:
- added joint LEFT_ARM_TO_LEFT_HAND_CONNECTOR: type fixed, parent left_ee, child left_base_link, origin xyz=0 0 0 rpy=0 0 0
- added joint LEFT_BASE_OFFSET: type fixed, parent left_hand_base_link, child left_base_offset, origin xyz=0 0.0298242 0 rpy=-0.0698132 0 0
- added joint LEFT_CONNECTOR: type fixed, parent left_base_link, child left_connector_link, origin xyz=0 0 0 rpy=1.5707963267948966 0 3.141592653589793
- added joint LEFT_HAND_BASE: type fixed, parent left_connector_link, child left_hand_base_link, origin xyz=0 0 0.002 rpy=0 0 0
- added joint LEFT_IF_DIP: type revolute, parent left_if_mcp_pitch_link, child left_if_dip_link, origin xyz=0 0.035 0 rpy=0.19353 0 0, axis 1 0 0, limit lower=0 upper=2.0944 effort=0 velocity=0, mimic joint=LEFT_IF_MCP_PITCH multiplier=1.2 offset=0.19373154697137057
- added joint LEFT_IF_MCP_PITCH: type revolute, parent left_base_offset, child left_if_mcp_pitch_link, origin xyz=-0.029003 0.088291 0.0022155 rpy=-0.029415 0.05236 0.034907, axis 1 0 0, limit lower=0 upper=1.309 effort=0 velocity=0
- added joint LEFT_LF_DIP: type revolute, parent left_lf_mcp_pitch_link, child left_lf_dip_link, origin xyz=0 0.035 0 rpy=0.20294 0 0, axis 1 0 0, limit lower=0 upper=2.0944 effort=0 velocity=0, mimic joint=LEFT_LF_MCP_PITCH multiplier=1.2 offset=0.20245819323134223
- added joint LEFT_LF_MCP_PITCH: type revolute, parent left_base_offset, child left_lf_mcp_pitch_link, origin xyz=0.033731 0.083777 0.0022155 rpy=-0.024909 -0.05236 -0.069813, axis 1 0 0, limit lower=0 upper=1.309 effort=0 velocity=0
- added joint LEFT_MF_DIP: type revolute, parent left_mf_mcp_pitch_link, child left_mf_dip_link, origin xyz=0 0.042 0 rpy=0.18357 0 0, axis 1 0 0, limit lower=0 upper=2.0944 effort=0 velocity=0, mimic joint=LEFT_MF_MCP_PITCH multiplier=1.2 offset=0.1832595714594046
- added joint LEFT_MF_MCP_PITCH: type revolute, parent left_base_offset, child left_mf_mcp_pitch_link, origin xyz=-0.008 0.092284 -0.0017707 rpy=0 0 0, axis 1 0 0, limit lower=0 upper=1.309 effort=0 velocity=0
- added joint LEFT_RF_DIP: type revolute, parent left_rf_mcp_pitch_link, child left_rf_dip_link, origin xyz=0 0.042 0 rpy=0.16583 0 0, axis 1 0 0, limit lower=0 upper=2.0944 effort=0 velocity=0, mimic joint=LEFT_RF_MCP_PITCH multiplier=1.2 offset=0.16580627893946132
- added joint LEFT_RF_MCP_PITCH: type revolute, parent left_base_offset, child left_rf_mcp_pitch_link, origin xyz=0.013103 0.090291 -0.0017845 rpy=-0.0092374 -0.05236 -0.034907, axis 1 0 0, limit lower=0 upper=1.309 effort=0 velocity=0
- added joint LEFT_T_CMC_YAW: type revolute, parent left_base_offset, child left_t_cmc_yaw_link, origin xyz=-0.0245 0.022632 0.023263 rpy=0.14578 -1.0699 -0.12808, axis 0 1 0, limit lower=0 upper=1.5708 effort=0 velocity=0
- added joint LEFT_T_MCP: type revolute, parent left_t_cmc_yaw_link, child left_t_mcp_link, origin xyz=0 0 0.013647 rpy=0.87266 -0.49642 0, axis -1 0 0, limit lower=0 upper=0.8727 effort=0 velocity=0
- added joint RIGHT_ARM_TO_RIGHT_HAND_CONNECTOR: type fixed, parent right_ee, child right_base_link, origin xyz=0 0 0 rpy=0 0 0
- added joint RIGHT_BASE_OFFSET: type fixed, parent right_hand_base_link, child right_base_offset, origin xyz=0 0.0298242 0 rpy=0 0 0
- added joint RIGHT_CONNECTOR: type fixed, parent right_base_link, child right_connector_link, origin xyz=0 0 0 rpy=1.5707963267948966 0 0
- added joint RIGHT_HAND_BASE: type fixed, parent right_connector_link, child right_hand_base_link, origin xyz=0 0 0.002 rpy=0 0 0
- added joint RIGHT_IF_DIP: type revolute, parent right_if_mcp_pitch_link, child right_if_dip_link, origin xyz=0 0.035 0 rpy=0.19353 0 0, axis 1 0 0, limit lower=0 upper=2.0944 effort=0 velocity=0, mimic joint=RIGHT_IF_MCP_PITCH multiplier=1.2 offset=0.19373154697137057
- added joint RIGHT_IF_MCP_PITCH: type revolute, parent right_base_offset, child right_if_mcp_pitch_link, origin xyz=0.029003 0.088231 -0.0039488 rpy=-0.09929 -0.054667 -0.031168, axis 1 0 0, limit lower=0 upper=1.309 effort=0 velocity=0
- added joint RIGHT_LF_DIP: type revolute, parent right_lf_mcp_pitch_link, child right_lf_dip_link, origin xyz=0 0.035 0 rpy=0.20294 0 0, axis 1 0 0, limit lower=0 upper=2.0944 effort=0 velocity=0, mimic joint=RIGHT_LF_MCP_PITCH multiplier=1.2 offset=0.20245819323134223
- added joint RIGHT_LF_MCP_PITCH: type revolute, parent right_base_offset, child right_lf_mcp_pitch_link, origin xyz=-0.033731 0.083727 -0.0036339 rpy=-0.094666 0.057099 0.065996, axis 1 0 0, limit lower=0 upper=1.309 effort=0 velocity=0
- added joint RIGHT_MF_DIP: type revolute, parent right_mf_mcp_pitch_link, child right_mf_dip_link, origin xyz=0 0.042 0 rpy=0.18357 0 0, axis 1 0 0, limit lower=0 upper=2.0944 effort=0 velocity=0, mimic joint=RIGHT_MF_MCP_PITCH multiplier=1.2 offset=0.1832595714594046
- added joint RIGHT_MF_MCP_PITCH: type revolute, parent right_base_offset, child right_mf_mcp_pitch_link, origin xyz=0.008 0.091935 -0.0082038 rpy=-0.069813 0 0, axis 1 0 0, limit lower=0 upper=1.309 effort=0 velocity=0
- added joint RIGHT_RF_DIP: type revolute, parent right_rf_mcp_pitch_link, child right_rf_dip_link, origin xyz=0 0.042 0 rpy=0.16583 0 0, axis 1 0 0, limit lower=0 upper=2.0944 effort=0 velocity=0, mimic joint=RIGHT_RF_MCP_PITCH multiplier=1.2 offset=0.16580627893946132
- added joint RIGHT_RF_MCP_PITCH: type revolute, parent right_base_offset, child right_rf_mcp_pitch_link, origin xyz=-0.013103 0.089947 -0.0080786 rpy=-0.079113 0.054667 0.031168, axis 1 0 0, limit lower=0 upper=1.309 effort=0 velocity=0
- added joint RIGHT_T_CMC_YAW: type revolute, parent right_base_offset, child right_t_cmc_yaw_link, origin xyz=0.0245 0.0242 0.021628 rpy=0 -0.49642 0, axis 0 -1 0, limit lower=0 upper=1.5708 effort=0 velocity=0
- added joint RIGHT_T_MCP: type revolute, parent right_t_cmc_yaw_link, child right_t_mcp_link, origin xyz=0.013647 0 0 rpy=-0.39332 0.31115 -0.93514, axis 0 0 1, limit lower=0 upper=0.87266 effort=0 velocity=0
